File: KICAD/first/first.kicad_pcb (KiCad board)
At the start: 2 copper layers, 140.5 x 334.5 mm, 216 parts, among them J1 SS-101-S-22, J2 SS-101-S-22, J3 SS-101-S-22, J4 SS-101-S-22, SW1 SW_SPDT, SW2 SW_Push, SW3 SW_Push, SW4 SW_Push, SW5 SW_Push, SW6 SW_Push, U1 ESP32-DEVKITC-32D, U2 74HC594, U3 74HC594, U4 74HC594

Commit message: pcb finished
add some holes for case to be attached
Parts:
- moved SW3 121.4 mm to (45.8, 202.5)
- moved LS1 117.3 mm to (43.2, 166.0)
- moved SW1 116.7 mm to (62.5, 164.5)
- moved SW4 112.3 mm to (58.8, 188.0)
- moved SW5 97.9 mm to (113.8, 165.0)
- moved SW6 89.0 mm to (102.2, 185.5)
- moved SW2 68.0 mm to (32.8, 188.0)
Routing:
- net GND: track 167.8 -> 499.4 mm, vias 6 -> 7
- net /Clock 1: track 0.00 -> 318.2 mm, vias 0 -> 8
- net /Latch 1: track 0.00 -> 312.0 mm, vias 0 -> 6
- net +5V: track 128.5 -> 422.0 mm, vias 5 -> 2
- net /sda: track 0.00 -> 290.3 mm
- net /scl: track 0.00 -> 280.0 mm, vias 0 -> 2
- net /Data 1: track 0.00 -> 200.2 mm, vias 0 -> 1
- net /Speaker: track 0.00 -> 105.5 mm, vias 0 -> 1
- net /Rotate button: track 0.00 -> 81.1 mm, vias 0 -> 1
- net /Left button: track 0.00 -> 78.9 mm, vias 0 -> 2
- net /Pause button: track 0.00 -> 54.0 mm
- net Net-(U2-QH'): track 0.00 -> 50.2 mm, vias 0 -> 2
- net /Right button: track 0.00 -> 48.8 mm
- net /Down button: track 0.00 -> 48.7 mm, vias 0 -> 1
- net Net-(U3-QH'): track 0.00 -> 31.4 mm, vias 0 -> 2
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- added copper zone on B.Cu, net GND
- added copper zone on F.Cu, net GND
Other:
- board size 140.5 x 334.5 mm -> 115.5 x 315.5 mm
